File: boards/photon_board/photon_board.sch (KiCad schematic (older format))
At the start: 2 parts

Commit message: add custom lvds receiver symbol
Parts:
- added U? (x2): SN65LVDT34D, Package_SO:SOIC-8_3.9x4.9mm_P1.27mm, symbol photon_board:SN65LVDT34D
- J2: renamed from J?; footprint (none) -> Connector_Dsub:DSUB-15-HD_Female_Horizontal_P2.29x1.98mm_EdgePinOffset3.03mm_Housed_MountingHolesOffset4.94mm
- gave numbers to parts that had none: 1
Changed lines of the file:
@@
 EESchema Schematic File Version 4
+LIBS:photon_board-cache
 EELAYER 26 0
 EELAYER END
@@
 $EndDescr
 $Comp
-L Connector_Generic:Conn_02x20_Odd_Even J?
+L Connector_Generic:Conn_02x20_Odd_Even J1
 U 1 1 5BD9CB75
 P 1750 2050
-F 0 "J?" H 1800 3167 50  0000 C CNN
+F 0 "J1" H 1800 3167 50  0000 C CNN
 F 1 "TERASIC" H 1800 3076 50  0000 C CNN
 F 2 "Connector_PinSocket_2.54mm:PinSocket_2x20_P2.54mm_Vertical" H 1750 2050 50  0001 C CNN
@@
 NoConn ~ 1550 1250
 $Comp
-L power:+5V #PWR?
+L power:+5V #PWR0101
 U 1 1 5BD9CC1E
 P 1300 1650
-F 0 "#PWR?" H 1300 1500 50  0001 C CNN
+F 0 "#PWR0101" H 1300 1500 50  0001 C CNN
 F 1 "+5V" H 1315 1823 50  0000 C CNN
 F 2 "" H 1300 1650 50  0001 C CNN
@@
 	1300 1650 1550 1650
 $Comp
-L power:+3V3 #PWR?
+L power:+3V3 #PWR0102
 U 1 1 5BD9CCF3
 P 1300 2550
-F 0 "#PWR?" H 1300 2400 50  0001 C CNN
+F 0 "#PWR0102" H 1300 2400 50  0001 C CNN
 F 1 "+3V3" H 1315 2723 50  0000 C CNN
 F 2 "" H 1300 2550 50  0001 C CNN
@@
 	1300 2550 1550 2550
 $Comp
-L power:GND #PWR?
+L power:GND #PWR0103
 U 1 1 5BD9CD64
 P 2300 1650
-F 0 "#PWR?" H 2300 1400 50  0001 C CNN
+F 0 "#PWR0103" H 2300 1400 50  0001 C CNN
 F 1 "GND" H 2305 1477 50  0000 C CNN
 F 2 "" H 2300 1650 50  0001 C CNN
@@
 	2300 1650 2050 1650
 $Comp
-L power:GND #PWR?
+L power:GND #PWR0104
 U 1 1 5BD9CDEB
 P 2300 2550
-F 0 "#PWR?" H 2300 2300 50  0001 C CNN
+F 0 "#PWR0104" H 2300 2300 50  0001 C CNN
 F 1 "GND" H 2305 2377 50  0000 C CNN
 F 2 "" H 2300 2550 50  0001 C CNN
@@
 	2300 2550 2050 2550
 $Comp
-L Connector:DB15_Female_HighDensity_MountingHoles J?
+L Connector:DB15_Female_HighDensity_MountingHoles J2
 U 1 1 5BD9D048
-P 8100 1900
-F 0 "J?" H 8100 2767 50  0000 C CNN
-F 1 "PHOTON" H 8100 2676 50  0000 C CNN
-F 2 "" H 7150 2300 50  0001 C CNN
-F 3 " ~" H 7150 2300 50  0001 C CNN
-	1    8100 1900
+P 5650 2050
+F 0 "J2" H 5650 2917 50  0000 C CNN
+F 1 "PHOTON" H 5650 2826 50  0000 C CNN
+F 2 "Connector_Dsub:DSUB-15-HD_Female_Horizontal_P2.29x1.98mm_EdgePinOffset3.03mm_Housed_MountingHolesOffset4.94mm" H 4700 2450 50  0001 C CNN
+F 3 " ~" H 4700 2450 50  0001 C CNN
+	1    5650 2050
 	1    0    0    -1
 $EndComp
 $Comp
-L power:GND #PWR?
+L power:GND #PWR0105
 U 1 1 5BD9D12F
-P 8100 2600
-F 0 "#PWR?" H 8100 2350 50  0001 C CNN
-F 1 "GND" H 8105 2427 50  0000 C CNN
-F 2 "" H 8100 2600 50  0001 C CNN
-F 3 "" H 8100 2600 50  0001 C CNN
-	1    8100 2600
+P 5650 2750
+F 0 "#PWR0105" H 5650 2500 50  0001 C CNN
+F 1 "GND" H 5655 2577 50  0000 C CNN
+F 2 "" H 5650 2750 50  0001 C CNN
+F 3 "" H 5650 2750 50  0001 C CNN
+	1    5650 2750
 	1    0    0    -1
 $EndComp
-Text Label 7800 1500 2    50   ~ 0
+Text Label 5350 1650 2    50   ~ 0
 DATA_SYNC+
-Text Label 7800 1700 2    50   ~ 0
+Text Label 5350 1850 2    50   ~ 0
 DATA1_OUT+
-Text Label 7800 1900 2    50   ~ 0
+Text Label 5350 2050 2    50   ~ 0
 DATA2_OUT+
-Text Label 7800 2100 2    50   ~ 0
+Text Label 5350 2250 2    50   ~ 0
 DATA_CLK+
-Text Label 7800 1400 2    50   ~ 0
+Text Label 5350 1550 2    50   ~ 0
 DATA_SYNC-
-Text Label 7800 1600 2    50   ~ 0
+Text Label 5350 1750 2    50   ~ 0
 DATA1_OUT-
-Text Label 7800 1800 2    50   ~ 0
+Text Label 5350 1950 2    50   ~ 0
 DATA2_OUT-
-Text Label 7800 2000 2    50   ~ 0
+Text Label 5350 2150 2    50   ~ 0
 DATA_CLK-
 $Comp
-L power:GND #PWR?
+L power:GND #PWR0106
 U 1 1 5BD9D377
-P 7450 2200
-F 0 "#PWR?" H 7450 1950 50  0001 C CNN
-F 1 "GND" H 7455 2027 50  0000 C CNN
-F 2 "" H 7450 2200 50  0001 C CNN
-F 3 "" H 7450 2200 50  0001 C CNN
-	1    7450 2200
+P 5000 2350
+F 0 "#PWR0106" H 5000 2100 50  0001 C CNN
+F 1 "GND" H 5005 2177 50  0000 C CNN
+F 2 "" H 5000 2350 50  0001 C CNN
+F 3 "" H 5000 2350 50  0001 C CNN
+	1    5000 2350
 	1    0    0    -1
 $EndComp
 Wire Wire Line
-	7450 2200 7800 2200
-NoConn ~ 7800 2300
-NoConn ~ 8400 1900
-NoConn ~ 8400 2100
-NoConn ~ 8400 2300
+	5000 2350 5350 2350
+NoConn ~ 5350 2450
+NoConn ~ 5950 2050
+NoConn ~ 5950 2250
+NoConn ~ 5950 2450
+$Comp
+L photon_board:SN65LVDT34D U?
+U 1 1 5BDA5F0C
+P 3450 1450
+F 0 "U?" H 3450 2228 50  0000 C CNN
+F 1 "SN65LVDT34D" H 3450 2137 50  0000 C CNN
+F 2 "Package_SO:SOIC-8_3.9x4.9mm_P1.27mm" H 3400 800 50  0001 C CNN
+F 3 "https://www.digikey.com/product-detail/en/texas-instruments/SN65LVDT34D/296-9751-5-ND/380393" H 2750 600 50  0001 C CNN
+	1    3450 1450
+	-1   0    0    -1
+$EndComp
+$Comp
+L photon_board:SN65LVDT34D U?
+U 1 1 5BDA6017
+P 3450 3000
+F 0 "U?" H 3450 3778 50  0000 C CNN
+F 1 "SN65LVDT34D" H 3450 3687 50  0000 C CNN
+F 2 "Package_SO:SOIC-8_3.9x4.9mm_P1.27mm" H 3400 2350 50  0001 C CNN
+F 3 "https://www.digikey.com/product-detail/en/texas-instruments/SN65LVDT34D/296-9751-5-ND/380393" H 2750 2150 50  0001 C CNN
+	1    3450 3000
+	-1   0    0    -1
+$EndComp
 $EndSCHEMATC

Commit message: finalize schematic
Parts:
- added C1, C3: 1u, Capacitor_SMD:C_0603_1608Metric_Pad1.05x0.95mm_HandSolder, symbol Device:C_Small
- added C2, C4: 0.1u, Capacitor_SMD:C_0603_1608Metric_Pad1.05x0.95mm_HandSolder, symbol Device:C_Small
- gave numbers to parts that had none: 2
Connections:
- net labels added: DATA1_OUT, DATA2_OUT, DATA_CLK, DATA_SYNC
- wire segments 5 -> 15

Commit message: add connector for photon and make appropriate footprint
Parts:
- J2: footprint Connector_Dsub:DSUB-15-HD_Female_Horizontal_P2.29x1.98mm_EdgePinOffset3.03mm_Housed_MountingHolesOffset4.94mm -> d_connector:DSUB-15-HD_Female_Horizontal_Pitch2.28x2.54mm_EdgePinOffset8.89mm_Housed_MountingHolesOffset11.43mm
Changed lines of the file:
@@
 F 0 "J2" H 7150 2917 50  0000 C CNN
 F 1 "PHOTON" H 7150 2826 50  0000 C CNN
-F 2 "Connector_Dsub:DSUB-15-HD_Female_Horizontal_P2.29x1.98mm_EdgePinOffset3.03mm_Housed_MountingHolesOffset4.94mm" H 6200 2450 50  0001 C CNN
-F 3 " ~" H 6200 2450 50  0001 C CNN
+F 2 "d_connector:DSUB-15-HD_Female_Horizontal_Pitch2.28x2.54mm_EdgePinOffset8.89mm_Housed_MountingHolesOffset11.43mm" H 6200 2450 50  0001 C CNN
+F 3 "https://www.digikey.com/product-detail/en/amphenol-fci/ICD15S13E4GX00LF/609-5181-ND/1536501" H 6200 2450 50  0001 C CNN
 	1    7150 2050
 	1    0    0    -1

Commit message: add data out connector for eg logic analysis
Parts:
- added J3: DATA, Connector_PinHeader_2.54mm:PinHeader_1x06_P2.54mm_Vertical, symbol Connector_Generic:Conn_01x06
Changed lines of the file:
@@
 Text Label 3050 2150 2    50   ~ 0
 DATA_SYNC
+$Comp
+L Connector_Generic:Conn_01x06 J3
+U 1 1 5BF4356F
+P 4200 3000
+F 0 "J3" H 4279 2992 50  0000 L CNN
+F 1 "DATA" H 4279 2901 50  0000 L CNN
+F 2 "Connector_PinHeader_2.54mm:PinHeader_1x06_P2.54mm_Vertical" H 4200 3000 50  0001 C CNN
+F 3 "~" H 4200 3000 50  0001 C CNN
+	1    4200 3000
+	1    0    0    -1
+$EndComp
+$Comp
+L power:GND #PWR0107
+U 1 1 5BF4368D
+P 4000 2800
+F 0 "#PWR0107" H 4000 2550 50  0001 C CNN
+F 1 "GND" H 4005 2627 50  0000 C CNN
+F 2 "" H 4000 2800 50  0001 C CNN
+F 3 "" H 4000 2800 50  0001 C CNN
+	1    4000 2800
+	-1   0    0    1
+$EndComp
+Text Label 4000 2900 2    50   ~ 0
+DATA_CLK
+Text Label 4000 3000 2    50   ~ 0
+DATA2_OUT
+Text Label 4000 3100 2    50   ~ 0
+DATA1_OUT
+Text Label 4000 3200 2    50   ~ 0
+DATA_SYNC
+$Comp
+L power:GND #PWR0108
+U 1 1 5BF43968
+P 4000 3300
+F 0 "#PWR0108" H 4000 3050 50  0001 C CNN
+F 1 "GND" H 4005 3127 50  0000 C CNN
+F 2 "" H 4000 3300 50  0001 C CNN
+F 3 "" H 4000 3300 50  0001 C CNN
+	1    4000 3300
+	1    0    0    -1
+$EndComp
 $EndSCHEMATC
